File: hardware/joint_bench/joint_bench.kicad_sch (KiCad schematic)
At the start: 8 parts, among them J1 IMU GY-87, J2 Logic analyzer, J3 Test points, U1 WeAct BlackPill F411CEU6

Commit message: docs(hardware): switch the stage-A bench from the GY-87 to a GY-521
The GY-521 carries only an MPU-6050, so i2cscan now expects 68 alone. It has
no 3.3 V pin and no FSYNC pin, so the runbook's pull-up check reads the
resistor code or measures at the regulator, and the FSYNC bridge is gone.

Regenerate the KiCad files, which also clears the stale F411 part label.

Co-Authored-By: Claude Opus 5.5 <noreply@anthropic.com>
Parts:
- J1: value IMU GY-87 -> IMU GY-521
- U1: value WeAct BlackPill F411CEU6 -> WeAct BlackPill F401CEU6
Other:
- note added: "GY-521 cable, 30-60 cm: J1 VCC to VCC, GND to GND, SCL to SCL, SDA to SDA, INT to INT."
- note added: "Leave the GY-521's XDA, XCL and AD0 unconnected. Twist SCL with GND, SDA with VCC."
- note removed: "GY-87 cable, 30-60 cm: J1 VCC to VCC_IN, GND to GND, SCL to SCL, SDA to SDA, INT to INTA."
- note removed: "Tie the GY-87's FSYNC pin to its GND at the module end. Twist SCL with GND, SDA with VCC."
Changed lines of the file:
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@@
         (font
           (size 1.27 1.27))))
-    (property "Value" "WeAct BlackPill F411CEU6"
+    (property "Value" "WeAct BlackPill F401CEU6"
       (at 63.5 118.11 0)
       (effects
@@
         (font
           (size 1.27 1.27))))
-    (property "Value" "IMU GY-87"
+    (property "Value" "IMU GY-521"
       (at 177.8 48.26 0)
       (effects
@@
       (justify left bottom))
 )
-  (text "GY-87 cable, 30-60 cm: J1 VCC to VCC_IN, GND to GND, SCL to SCL, SDA to SDA, INT to INTA."
+  (text "GY-521 cable, 30-60 cm: J1 VCC to VCC, GND to GND, SCL to SCL, SDA to SDA, INT to INT."
     (exclude_from_sim no)
     (at 20.32 180.34 0)
@@
       (justify left bottom))
 )
-  (text "Tie the GY-87's FSYNC pin to its GND at the module end. Twist SCL with GND, SDA with VCC."
+  (text "Leave the GY-521's XDA, XCL and AD0 unconnected. Twist SCL with GND, SDA with VCC."
     (exclude_from_sim no)
     (at 20.32 187.96 0)
