File: hardware/joint_bench/trial_6x9.kicad_pcb (KiCad board)
At the start: 2 copper layers, 88.8 x 58.3 mm, 8 parts, among them J1 IMU GY-87, J2 Logic analyzer, J3 Test points, U1 WeAct BlackPill F411CEU6

Commit message: docs(hardware): switch the stage-A bench from the GY-87 to a GY-521
The GY-521 carries only an MPU-6050, so i2cscan now expects 68 alone. It has
no 3.3 V pin and no FSYNC pin, so the runbook's pull-up check reads the
resistor code or measures at the regulator, and the FSYNC bridge is gone.

Regenerate the KiCad files, which also clears the stale F411 part label.

Co-Authored-By: Claude Opus 5.5 <noreply@anthropic.com>
Parts:
- J1: value IMU GY-87 -> IMU GY-521
- U1: value WeAct BlackPill F411CEU6 -> WeAct BlackPill F401CEU6
Changed lines of the file:
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@@
           (thickness 0.15))
         (justify left)))
-    (property "Value" "WeAct BlackPill F411CEU6"
+    (property "Value" "WeAct BlackPill F401CEU6"
       (at -2.37 19.07 0)
       (layer "F.Fab")
@@
           (thickness 0.15))
         (justify left)))
-    (property "Value" "IMU GY-87"
+    (property "Value" "IMU GY-521"
       (at -1.27 12.43 0)
       (layer "F.Fab")
